Commit message: rubric: *Robot Model: 	  -Create a mobile robot model wth a RGBD camera and a laser sensor. 	  -Setup the Gazebo and Rviz environments and launch the robot inside the environment. 	  -The provided transform tree has proper linkages.
	*Mapping:
	  -Create the appropriate launch files such as: mapping and teleop

File: catkin_ws/src/udacity_map/urdf/ucho_bot.xacro (robot description, xacro)
@@ -213,5 +213,5 @@
     </visual>
   </link>
-  <joint type="fixed" name="camera_joint" >
+  <joint type="fixed" name="camera_link" >
     <origin xyz="0.25 0 0.1" rpy="0 0 0" />
     <child link="camera" />
@@ -243,4 +243,11 @@
     </visual>
   </link>
+<!--Joint-->
+  <joint name="camera_joint" type="fixed">
+      <origin xyz="0 0 0" rpy="-1.5707 0 -1.5707"/>
+      <parent link="camera"/>
+      <child link="camera_rgbd_frame"/>
+  </joint>
+<link name="camera_rgbd_frame"/>
   <joint type="fixed" name="hokuyo_joint" >
     <origin xyz="0.20 0 0.25" />
